File: PCB/RaspberryPiHat_V2/RPHat_V2/Hall Effect Schematics.sch (KiCad schematic (older format))
At the start: 4 parts

Commit message: Schematic clean-up
Changed lines of the file:
@@
 encoding utf-8
 Sheet 3 4
-Title ""
-Date ""
-Rev ""
+Title "Hall effect subcircuit"
+Date "2021-05-15"
+Rev "0.1"
 Comp ""
 Comment1 ""
@@
 U 1 1 6098D710
 P 1800 1400
-F 0 "U?" H 1570 1446 50  0000 R CNN
-F 1 "AH1806-P" H 1570 1355 50  0000 R CNN
+F 0 "U?" H 1570 1654 50  0000 R CNN
+F 1 "AH1806-P" H 1570 1575 50  0000 R CNN
 F 2 "Connector_PinHeader_2.54mm:PinHeader_1x03_P2.54mm_Vertical" H 1800 1400 50  0001 C CNN
 F 3 "https://www.diodes.com/assets/Datasheets/AH1806.pdf" H 1800 1400 50  0001 C CNN
@@
 P 1800 2000
 F 0 "#PWR?" H 1800 1750 50  0001 C CNN
-F 1 "GNDREF" H 1805 1827 50  0000 C CNN
+F 1 "GNDREF" H 1805 1827 50  0001 C CNN
 F 2 "" H 1800 2000 50  0001 C CNN
 F 3 "" H 1800 2000 50  0001 C CNN
@@
 P 2850 1750
 F 0 "#PWR?" H 2850 1500 50  0001 C CNN
-F 1 "GNDREF" V 2855 1622 50  0000 R CNN
+F 1 "GNDREF" V 2855 1622 50  0001 R CNN
 F 2 "" H 2850 1750 50  0001 C CNN
 F 3 "" H 2850 1750 50  0001 C CNN

Commit message: Started routing PCB
Parts:
- gave numbers to parts that had none: 4
Changed lines of the file:
@@
 $EndDescr
 $Comp
-L Sensor_Magnetic:AH1806-P U?
+L Sensor_Magnetic:AH1806-P U5
 U 1 1 6098D710
 P 1800 1400
-F 0 "U?" H 1570 1654 50  0000 R CNN
+F 0 "U5" H 1570 1654 50  0000 R CNN
 F 1 "AH1806-P" H 1570 1575 50  0000 R CNN
 F 2 "Connector_PinHeader_2.54mm:PinHeader_1x03_P2.54mm_Vertical" H 1800 1400 50  0001 C CNN
@@
 $EndComp
 $Comp
-L power:GNDREF #PWR?
+L power:GNDREF #PWR0139
 U 1 1 6098DD81
 P 1800 2000
-F 0 "#PWR?" H 1800 1750 50  0001 C CNN
+F 0 "#PWR0139" H 1800 1750 50  0001 C CNN
 F 1 "GNDREF" H 1805 1827 50  0001 C CNN
 F 2 "" H 1800 2000 50  0001 C CNN
@@
 $EndComp
 $Comp
-L power:+3.3V #PWR?
+L power:+3.3V #PWR0140
 U 1 1 6098E018
 P 1800 850
-F 0 "#PWR?" H 1800 700 50  0001 C CNN
+F 0 "#PWR0140" H 1800 700 50  0001 C CNN
 F 1 "+3.3V" H 1815 1023 50  0000 C CNN
 F 2 "" H 1800 850 50  0001 C CNN
@@
 $EndComp
 $Comp
-L Device:C C?
+L Device:C C13
 U 1 1 6098E664
 P 1050 1450
-F 0 "C?" H 935 1404 50  0000 R CNN
+F 0 "C13" H 935 1404 50  0000 R CNN
 F 1 "100nF" H 935 1495 50  0000 R CNN
 F 2 "Capacitor_SMD:C_0805_2012Metric_Pad1.18x1.45mm_HandSolder" H 1088 1300 50  0001 C CNN
@@
 $EndComp
 $Comp
-L Device:R R?
+L Device:R R9
 U 1 1 6098F759
 P 2250 1150
-F 0 "R?" H 2320 1196 50  0000 L CNN
+F 0 "R9" H 2320 1196 50  0000 L CNN
 F 1 "100k" H 2320 1105 50  0000 L CNN
 F 2 "Resistor_SMD:R_0805_2012Metric_Pad1.20x1.40mm_HandSolder" V 2180 1150 50  0001 C CNN
@@
 	2250 1400 2300 1400
 $Comp
-L Connector_Generic:Conn_01x03 J?
+L Connector_Generic:Conn_01x03 J4
 U 1 1 60990D01
 P 3200 1750
-F 0 "J?" H 3280 1792 50  0000 L CNN
+F 0 "J4" H 3280 1792 50  0000 L CNN
 F 1 "Conn_01x03" H 3280 1701 50  0000 L CNN
 F 2 "Connector_PinHeader_2.54mm:PinHeader_1x03_P2.54mm_Vertical" H 3200 1750 50  0001 C CNN
@@
 OUTPUT
 $Comp
-L power:GNDREF #PWR?
+L power:GNDREF #PWR0141
 U 1 1 60991611
 P 2850 1750
-F 0 "#PWR?" H 2850 1500 50  0001 C CNN
+F 0 "#PWR0141" H 2850 1500 50  0001 C CNN
 F 1 "GNDREF" V 2855 1622 50  0001 R CNN
 F 2 "" H 2850 1750 50  0001 C CNN
@@
 $EndComp
 $Comp
-L power:+3.3V #PWR?
+L power:+3.3V #PWR0142
 U 1 1 60991D41
 P 2850 1850
-F 0 "#PWR?" H 2850 1700 50  0001 C CNN
+F 0 "#PWR0142" H 2850 1700 50  0001 C CNN
 F 1 "+3.3V" V 2865 1978 50  0000 L CNN
 F 2 "" H 2850 1850 50  0001 C CNN

Commit message: Added footprints to all componetns
Parts:
- C13: footprint Capacitor_SMD:C_0805_2012Metric_Pad1.18x1.45mm_HandSolder -> Capacitor_SMD:C_0603_1608Metric_Pad1.08x0.95mm_HandSolder
- R9: footprint Resistor_SMD:R_0805_2012Metric_Pad1.20x1.40mm_HandSolder -> Resistor_SMD:R_0603_1608Metric_Pad0.98x0.95mm_HandSolder
Changed lines of the file:
@@
 F 0 "C13" H 935 1404 50  0000 R CNN
 F 1 "100nF" H 935 1495 50  0000 R CNN
-F 2 "Capacitor_SMD:C_0805_2012Metric_Pad1.18x1.45mm_HandSolder" H 1088 1300 50  0001 C CNN
+F 2 "Capacitor_SMD:C_0603_1608Metric_Pad1.08x0.95mm_HandSolder" H 1088 1300 50  0001 C CNN
 F 3 "~" H 1050 1450 50  0001 C CNN
 	1    1050 1450
@@
 F 0 "R9" H 2320 1196 50  0000 L CNN
 F 1 "100k" H 2320 1105 50  0000 L CNN
-F 2 "Resistor_SMD:R_0805_2012Metric_Pad1.20x1.40mm_HandSolder" V 2180 1150 50  0001 C CNN
+F 2 "Resistor_SMD:R_0603_1608Metric_Pad0.98x0.95mm_HandSolder" V 2180 1150 50  0001 C CNN
 F 3 "~" H 2250 1150 50  0001 C CNN
 	1    2250 1150
