File: PCB/RaspberryPiHat_V2/RPHat_V2/RPHat_V2.sch (KiCad schematic (older format))
At the start: 14 parts

Commit message: Working on the PCB
Parts:
- added BT?: Battery, Connector_PinSocket_2.00mm:PinSocket_1x02_P2.00mm_Vertical, symbol Device:Battery
Connections:
- net labels added: PWM_Left, PWM_Right
- wire segments 66 -> 70
Changed lines of the file:
@@
 F1 "Servos_Motors.sch" 50
 $EndSheet
+Text GLabel 3850 6250 2    50   Input ~ 0
+PWM_Right
+Text GLabel 3850 5750 2    50   Input ~ 0
+PWM_Left
+Wire Wire Line
+	3850 5750 3650 5750
+Wire Wire Line
+	3850 6250 3650 6250
+$Comp
+L Device:Battery BT?
+U 1 1 60A0D572
+P 850 3350
+F 0 "BT?" H 958 3396 50  0000 L CNN
+F 1 "Battery" H 958 3305 50  0000 L CNN
+F 2 "Connector_PinSocket_2.00mm:PinSocket_1x02_P2.00mm_Vertical" V 850 3410 50  0001 C CNN
+F 3 "~" V 850 3410 50  0001 C CNN
+	1    850  3350
+	1    0    0    -1
+$EndComp
+$Comp
+L power:+BATT #PWR?
+U 1 1 60A138F9
+P 850 3000
+F 0 "#PWR?" H 850 2850 50  0001 C CNN
+F 1 "+BATT" H 865 3173 50  0000 C CNN
+F 2 "" H 850 3000 50  0001 C CNN
+F 3 "" H 850 3000 50  0001 C CNN
+	1    850  3000
+	1    0    0    -1
+$EndComp
+Wire Wire Line
+	850  3150 850  3000
+$Comp
+L power:GNDREF #PWR?
+U 1 1 60A18EAA
+P 850 3700
+F 0 "#PWR?" H 850 3450 50  0001 C CNN
+F 1 "GNDREF" H 855 3527 50  0000 C CNN
+F 2 "" H 850 3700 50  0001 C CNN
+F 3 "" H 850 3700 50  0001 C CNN
+	1    850  3700
+	1    0    0    -1
+$EndComp
+Wire Wire Line
+	850  3550 850  3700
 $EndSCHEMATC

Commit message: Configured pinout for logic converter
Parts:
- PS?: symbol RPMB5.0-3.0:RPMB5.0-3.0 -> RPHat_V2-rescue:RPMB5.0-3.0-RPMB5.0-3.0
- U?: symbol teensy:Teensy4.0 -> RPHat_V2-rescue:Teensy4.0-teensy
Changed lines of the file:
@@
 $EndDescr
 $Comp
-L RPMB5.0-3.0:RPMB5.0-3.0 PS?
+L RPHat_V2-rescue:RPMB5.0-3.0-RPMB5.0-3.0 PS?
 U 1 1 608338A4
 P 2200 1250
@@
 $EndComp
 $Comp
-L teensy:Teensy4.0 U?
+L RPHat_V2-rescue:Teensy4.0-teensy U?
 U 1 1 608349BD
 P 8050 2350

Commit message: Started routing for the BMS
Connections:
- net labels added: -BATT, BME_CS_33, IMU_CS_33, SPI_CLK_33, SPI_MISO_33, SPI_MOSI_33
- wire segments 70 -> 75
Changed lines of the file:
@@
 F1 "Servos_Motors.sch" 50
 $EndSheet
-Text GLabel 3850 6250 2    50   Input ~ 0
+Text GLabel 6750 1600 0    50   Input ~ 0
 PWM_Right
-Text GLabel 3850 5750 2    50   Input ~ 0
+Text GLabel 6750 2000 0    50   Input ~ 0
 PWM_Left
 Wire Wire Line
-	3850 5750 3650 5750
+	6750 2000 6950 2000
 Wire Wire Line
-	3850 6250 3650 6250
+	6750 1600 6950 1600
 $Comp
 L Device:Battery BT?
@@
 Wire Wire Line
 	850  3150 850  3000
+Text GLabel 3800 6250 2    50   Input ~ 0
+SPI_MISO_33
+Text GLabel 3800 6350 2    50   Input ~ 0
+SPI_MOSI_33
+Text GLabel 3800 6450 2    50   Input ~ 0
+SPI_CLK_33
+Text GLabel 3750 6650 2    50   Input ~ 0
+IMU_CS_33
+Text GLabel 3750 6750 2    50   Input ~ 0
+BME_CS_33
+Wire Wire Line
+	3800 6250 3650 6250
+Wire Wire Line
+	3800 6350 3650 6350
+Wire Wire Line
+	3800 6450 3650 6450
+Wire Wire Line
+	3750 6650 3650 6650
+Wire Wire Line
+	3750 6750 3650 6750
 $Comp
-L power:GNDREF #PWR?
-U 1 1 60A18EAA
-P 850 3700
-F 0 "#PWR?" H 850 3450 50  0001 C CNN
-F 1 "GNDREF" H 855 3527 50  0000 C CNN
-F 2 "" H 850 3700 50  0001 C CNN
-F 3 "" H 850 3700 50  0001 C CNN
-	1    850  3700
-	1    0    0    -1
+L power:-BATT #PWR?
+U 1 1 60A01C3B
+P 850 3800
+F 0 "#PWR?" H 850 3650 50  0001 C CNN
+F 1 "-BATT" H 865 3973 50  0000 C CNN
+F 2 "" H 850 3800 50  0001 C CNN
+F 3 "" H 850 3800 50  0001 C CNN
+	1    850  3800
+	-1   0    0    1
 $EndComp
 Wire Wire Line
-	850  3550 850  3700
+	850  3550 850  3800
 $EndSCHEMATC

Commit message: Continued routing the pcb. Added current sensing sensor
Parts:
- added R? (x2): TBU, Resistor_SMD:R_0603_1608Metric_Pad0.98x0.95mm_HandSolder, symbol Device:R
- R?: value R -> 4.7k
Connections:
- net labels added: +3V3, Neopixels_1, Neopixels_2, PWMservo_1, PWMservo_2, PWMservo_3, PWMservo_4, PWMservo_5, PWMservo_6, SCL, SDA, VCC
- net labels removed: -BATT
- wire segments 75 -> 117
Other:
- note added: "Pullups need to be calculated based \non slva689 application note from \ntexas instruments\n"

Commit message: Schematic clean-up
Parts:
- removed D?: LED, symbol Device:LED
- removed R?: 4.7k, symbol Device:R
- removed SW?: SW_DPDT_x2, symbol Switch:SW_DPDT_x2
- removed U?: Teensy4.0, symbol RPHat_V2-rescue:Teensy4.0-teensy
Other:
- moved on the sheet: BT?
Changed lines of the file:
@@
 encoding utf-8
 Sheet 1 4
-Title ""
-Date ""
-Rev ""
+Title "Rover PCB schematic"
+Date "2021-05-15"
+Rev "0.1"
 Comp ""
 Comment1 ""
@@
 $EndComp
 $Comp
-L RPHat_V2-rescue:Teensy4.0-teensy U?
-U 1 1 608349BD
-P 8050 2350
-F 0 "U?" H 8050 3965 50  0000 C CNN
-F 1 "Teensy4.0" H 8050 3874 50  0000 C CNN
-F 2 "" H 7650 2550 50  0001 C CNN
-F 3 "" H 7650 2550 50  0001 C CNN
-	1    8050 2350
-	1    0    0    -1
-$EndComp
-$Comp
 L Connector:Raspberry_Pi_2_3 J?
 U 1 1 608367C5
@@
 	1    0    0    -1
 $EndComp
-$Comp
-L Switch:SW_DPDT_x2 SW?
-U 1 1 60839FA9
-P 9450 3300
-F 0 "SW?" H 9450 3585 50  0000 C CNN
-F 1 "SW_DPDT_x2" H 9450 3494 50  0000 C CNN
-F 2 "" H 9450 3300 50  0001 C CNN
-F 3 "~" H 9450 3300 50  0001 C CNN
-	1    9450 3300
-	1    0    0    -1
-$EndComp
-$Comp
-L power:+5V #PWR?
-U 1 1 60850A7F
-P 9800 3100
-F 0 "#PWR?" H 9800 2950 50  0001 C CNN
-F 1 "+5V" H 9815 3273 50  0000 C CNN
-F 2 "" H 9800 3100 50  0001 C CNN
-F 3 "" H 9800 3100 50  0001 C CNN
-	1    9800 3100
-	1    0    0    -1
-$EndComp
-Wire Wire Line
-	9650 3200 9800 3200
-Wire Wire Line
-	9800 3200 9800 3100
-Wire Wire Line
-	9250 3300 9150 3300
 $Comp
 L Device:C C?
@@
 	3850 2200 3850 2250
 $Comp
-L Device:LED D?
-U 1 1 6088E6FB
-P 9400 3600
-F 0 "D?" V 9439 3482 50  0000 R CNN
-F 1 "LED" V 9348 3482 50  0000 R CNN
-F 2 "" H 9400 3600 50  0001 C CNN
-F 3 "~" H 9400 3600 50  0001 C CNN
-	1    9400 3600
-	-1   0    0    1
-$EndComp
-Connection ~ 9250 3300
-$Comp
-L Device:R R?
-U 1 1 60890E09
-P 9600 3800
-F 0 "R?" H 9670 3846 50  0000 L CNN
-F 1 "4.7k" H 9670 3755 50  0000 L CNN
-F 2 "" V 9530 3800 50  0001 C CNN
-F 3 "~" H 9600 3800 50  0001 C CNN
-	1    9600 3800
-	1    0    0    -1
-$EndComp
-Wire Wire Line
-	9600 3600 9600 3650
-$Comp
-L power:GNDREF #PWR?
-U 1 1 6089275F
-P 9600 4000
-F 0 "#PWR?" H 9600 3750 50  0001 C CNN
-F 1 "GNDREF" H 9605 3827 50  0001 C CNN
-F 2 "" H 9600 4000 50  0001 C CNN
-F 3 "" H 9600 4000 50  0001 C CNN
-	1    9600 4000
-	1    0    0    -1
-$EndComp
-Wire Wire Line
-	9600 3950 9600 4000
-Wire Wire Line
-	9250 3600 9250 3300
-Wire Wire Line
-	9550 3600 9600 3600
-$Comp
 L power:+5V #PWR?
 U 1 1 608B20C1
@@
 Wire Wire Line
 	2050 5150 1800 5150
-Text GLabel 6800 1100 0    50   Input ~ 0
-Teensy_Uart_RX
-Text GLabel 6800 1200 0    50   Input ~ 0
-Teensy_Uart_TX
-Wire Wire Line
-	6950 1100 6800 1100
-Wire Wire Line
-	6950 1200 6800 1200
 $Sheet
 S 7300 4700 1350 900
@@
 F1 "Servos_Motors.sch" 50
 $EndSheet
-Text GLabel 6750 1300 0    50   Input ~ 0
-PWM_Right
-Text GLabel 6750 1400 0    50   Input ~ 0
-PWM_Left
-Wire Wire Line
-	6750 1400 6950 1400
-Wire Wire Line
-	6750 1300 6950 1300
 $Comp
 L Device:Battery BT?
 U 1 1 60A0D572
-P 850 3350
-F 0 "BT?" H 958 3396 50  0000 L CNN
-F 1 "Battery" H 958 3305 50  0000 L CNN
-F 2 "Connector_PinSocket_2.00mm:PinSocket_1x02_P2.00mm_Vertical" V 850 3410 50  0001 C CNN
-F 3 "~" V 850 3410 50  0001 C CNN
-	1    850  3350
+P 800 2500
+F 0 "BT?" H 908 2546 50  0000 L CNN
+F 1 "Battery" H 908 2455 50  0000 L CNN
+F 2 "Connector_PinSocket_2.00mm:PinSocket_1x02_P2.00mm_Vertical" V 800 2560 50  0001 C CNN
+F 3 "~" V 800 2560 50  0001 C CNN
+	1    800  2500
 	1    0    0    -1
 $EndComp
@@
 L power:+BATT #PWR?
 U 1 1 60A138F9
-P 850 3000
-F 0 "#PWR?" H 850 2850 50  0001 C CNN
-F 1 "+BATT" H 865 3173 50  0000 C CNN
-F 2 "" H 850 3000 50  0001 C CNN
-F 3 "" H 850 3000 50  0001 C CNN
-	1    850  3000
-	1    0    0    -1
-$EndComp
-Wire Wire Line
-	850  3150 850  3000
+P 800 2150
+F 0 "#PWR?" H 800 2000 50  0001 C CNN
+F 1 "+BATT" H 815 2323 50  0000 C CNN
+F 2 "" H 800 2150 50  0001 C CNN
+F 3 "" H 800 2150 50  0001 C CNN
+	1    800  2150
+	1    0    0    -1
+$EndComp
+Wire Wire Line
+	800  2300 800  2150
 Text GLabel 3800 6250 2    50   Input ~ 0
 SPI_MISO_33
@@
 	1950 6150 2050 6150
 Wire Wire Line
-	850  3550 850  3800
+	800  2700 800  2950
 $Comp
 L power:VCC #PWR?
@@
 L power:GNDREF #PWR?
 U 1 1 60A67F58
-P 850 3800
-F 0 "#PWR?" H 850 3550 50  0001 C CNN
-F 1 "GNDREF" H 855 3627 50  0001 C CNN
-F 2 "" H 850 3800 50  0001 C CNN
-F 3 "" H 850 3800 50  0001 C CNN
-	1    850  3800
+P 800 2950
+F 0 "#PWR?" H 800 2700 50  0001 C CNN
+F 1 "GNDREF" H 805 2777 50  0001 C CNN
+F 2 "" H 800 2950 50  0001 C CNN
+F 3 "" H 800 2950 50  0001 C CNN
+	1    800  2950
 	1    0    0    -1
 $EndComp
@@
 Text Notes 3600 4500 0    50   ~ 0
 Pullups need to be calculated based \non slva689 application note from \ntexas instruments\n
-Text GLabel 6750 1500 0    50   Input ~ 0
-PWMservo_1
-Text GLabel 9300 2500 2    50   Input ~ 0
-Neopixels_1
-Text GLabel 6750 1600 0    50   Input ~ 0
-PWMservo_2
-Text GLabel 6750 1700 0    50   Input ~ 0
-PWMservo_3
-Text GLabel 6750 1800 0    50   Input ~ 0
-PWMservo_4
-Text GLabel 6750 1900 0    50   Input ~ 0
-PWMservo_5
-Text GLabel 6750 2000 0    50   Input ~ 0
-PWMservo_6
-Text GLabel 9300 2400 2    50   Input ~ 0
-Neopixels_2
-$Comp
-L power:GNDREF #PWR?
-U 1 1 60ADCEA9
-P 6850 1000
-F 0 "#PWR?" H 6850 750 50  0001 C CNN
-F 1 "GNDREF" H 6855 827 50  0001 C CNN
-F 2 "" H 6850 1000 50  0001 C CNN
-F 3 "" H 6850 1000 50  0001 C CNN
-	1    6850 1000
-	0    1    1    0
-$EndComp
-Wire Wire Line
-	6950 1000 6850 1000
 Wire Wire Line
 	1800 1550 2000 1550
-Wire Wire Line
-	6750 1500 6950 1500
-Wire Wire Line
-	6750 1600 6950 1600
-Wire Wire Line
-	6750 1700 6950 1700
-Wire Wire Line
-	6750 1800 6950 1800
-Wire Wire Line
-	6750 1900 6950 1900
-Wire Wire Line
-	6750 2000 6950 2000
-Wire Wire Line
-	9300 2400 9150 2400
-Wire Wire Line
-	9300 2500 9150 2500
 $EndSCHEMATC

Commit message: Started routing PCB
Parts:
- gave numbers to parts that had none: 13
Connections:
- net Teensy_Uart_RX renamed GPS_Uart_RX
- net Teensy_Uart_TX renamed GPS_Uart_TX
Changed lines of the file:
@@
 $EndDescr
 $Comp
-L RPHat_V2-rescue:RPMB5.0-3.0-RPMB5.0-3.0 PS?
+L RPHat_V2-rescue:RPMB5.0-3.0-RPMB5.0-3.0 PS1
 U 1 1 608338A4
 P 2200 1250
-F 0 "PS?" H 2850 1515 50  0000 C CNN
+F 0 "PS1" H 2850 1515 50  0000 C CNN
 F 1 "RPMB5.0-3.0" H 2850 1424 50  0000 C CNN
 F 2 "RPMB5030" H 3350 1350 50  0001 L CNN
@@
 $EndComp
 $Comp
-L Connector:Raspberry_Pi_2_3 J?
+L Connector:Raspberry_Pi_2_3 J1
 U 1 1 608367C5
 P 2850 5950
-F 0 "J?" H 2165 7431 50  0000 C CNN
+F 0 "J1" H 2165 7431 50  0000 C CNN
 F 1 "Raspberry_Pi_2_3" H 2165 7340 50  0000 C CNN
 F 2 "" H 2850 5950 50  0001 C CNN
@@
 $EndComp
 $Comp
-L Device:C C?
+L Device:C C3
 U 1 1 60855818
 P 1400 1400
-F 0 "C?" H 1515 1446 50  0000 L CNN
+F 0 "C3" H 1515 1446 50  0000 L CNN
 F 1 "10uF" H 1515 1355 50  0000 L CNN
 F 2 "Capacitor_SMD:C_1210_3225Metric_Pad1.33x2.70mm_HandSolder" H 1438 1250 50  0001 C CNN
@@
 $EndComp
 $Comp
-L Device:C C?
+L Device:C C2
 U 1 1 60856C0C
 P 1100 1400
-F 0 "C?" H 1215 1446 50  0000 L CNN
+F 0 "C2" H 1215 1446 50  0000 L CNN
 F 1 "10uF" H 1215 1355 50  0000 L CNN
 F 2 "Capacitor_SMD:C_1210_3225Metric_Pad1.33x2.70mm_HandSolder" H 1138 1250 50  0001 C CNN
@@
 $EndComp
 $Comp
-L Device:C C?
+L Device:C C1
 U 1 1 6085B575
 P 800 1400
-F 0 "C?" H 915 1446 50  0000 L CNN
+F 0 "C1" H 915 1446 50  0000 L CNN
 F 1 "10uF" H 915 1355 50  0000 L CNN
 F 2 "Capacitor_SMD:C_1210_3225Metric_Pad1.33x2.70mm_HandSolder" H 838 1250 50  0001 C CNN
@@
 $EndComp
 $Comp
-L power:GNDREF #PWR?
+L power:GNDREF #PWR0101
 U 1 1 6085D5E0
 P 800 1650
-F 0 "#PWR?" H 800 1400 50  0001 C CNN
+F 0 "#PWR0101" H 800 1400 50  0001 C CNN
 F 1 "GNDREF" H 805 1477 50  0001 C CNN
 F 2 "" H 800 1650 50  0001 C CNN
@@
 $EndComp
 $Comp
-L power:GNDREF #PWR?
+L power:GNDREF #PWR0102
 U 1 1 6085DEB3
 P 1100 1650
-F 0 "#PWR?" H 1100 1400 50  0001 C CNN
+F 0 "#PWR0102" H 1100 1400 50  0001 C CNN
 F 1 "GNDREF" H 1105 1477 50  0001 C CNN
 F 2 "" H 1100 1650 50  0001 C CNN
@@
 $EndComp
 $Comp
-L power:GNDREF #PWR?
+L power:GNDREF #PWR0103
 U 1 1 6085E1F0
 P 1400 1650
-F 0 "#PWR?" H 1400 1400 50  0001 C CNN
+F 0 "#PWR0103" H 1400 1400 50  0001 C CNN
 F 1 "GNDREF" H 1405 1477 50  0001 C CNN
 F 2 "" H 1400 1650 50  0001 C CNN
@@
 	1400 1550 1400 1650
 $Comp
-L pspice:INDUCTOR L?
+L pspice:INDUCTOR L1
 U 1 1 6085F0A3
 P 1700 1250
-F 0 "L?" H 1700 1465 50  0000 C CNN
+F 0 "L1" H 1700 1465 50  0000 C CNN
 F 1 "2.2uH" H 1700 1374 50  0000 C CNN
 F 2 "Inductor_SMD:L_1008_2520Metric_Pad1.43x2.20mm_HandSolder" H 1700 1250 50  0001 C CNN
@@
 $EndComp
 $Comp
-L Device:C C?
+L Device:C C4
 U 1 1 60862A5D
 P 2000 1400
-F 0 "C?" H 2115 1446 50  0000 L CNN
+F 0 "C4" H 2115 1446 50  0000 L CNN
 F 1 "C" H 2115 1355 50  0000 L CNN
 F 2 "Capacitor_SMD:C_1210_3225Metric_Pad1.33x2.70mm_HandSolder" H 2038 1250 50  0001 C CNN
@@
 	2100 1250 2200 1250
 $Comp
-L power:GNDREF #PWR?
+L power:GNDREF #PWR0104
 U 1 1 60862A63
 P 1800 1600
-F 0 "#PWR?" H 1800 1350 50  0001 C CNN
+F 0 "#PWR0104" H 1800 1350 50  0001 C CNN
 F 1 "GNDREF" H 1805 1427 50  0001 C CNN
 F 2 "" H 1800 1600 50  0001 C CNN
@@
 Connection ~ 2000 1550
 $Comp
-L power:+5V #PWR?
+L power:+5V #PWR0105
 U 1 1 6086D5CD
 P 2150 1650
-F 0 "#PWR?" H 2150 1500 50  0001 C CNN
+F 0 "#PWR0105" H 2150 1500 50  0001 C CNN
 F 1 "+5V" V 2165 1778 50  0000 L CNN
 F 2 "" H 2150 1650 50  0001 C CNN
@@
 	2200 1650 2150 1650
 $Comp
-L power:+5V #PWR?
+L power:+5V #PWR0106
 U 1 1 608702EB
 P 2150 2150
-F 0 "#PWR?" H 2150 2000 50  0001 C CNN
+F 0 "#PWR0106" H 2150 2000 50  0001 C CNN
 F 1 "+5V" V 2165 2278 50  0000 L CNN
 F 2 "" H 2150 2150 50  0001 C CNN
@@
 	2200 2150 2150 2150
 $Comp
-L power:GNDREF #PWR?
+L power:GNDREF #PWR0107
 U 1 1 60871C04
 P 1800 2100
-F 0 "#PWR?" H 1800 1850 50  0001 C CNN
+F 0 "#PWR0107" H 1800 1850 50  0001 C CNN
 F 1 "GNDREF" H 1805 1927 50  0001 C CNN
 F 2 "" H 1800 2100 50  0001 C CNN
@@
 Connection ~ 2050 2050
 $Comp
-L power:GNDREF #PWR?
+L power:GNDREF #PWR0108
 U 1 1 60875D28
 P 2000 2500
-F 0 "#PWR?" H 2000 2250 50  0001 C CNN
+F 0 "#PWR0108" H 2000 2250 50  0001 C CNN
 F 1 "GNDREF" H 2005 2327 50  0001 C CNN
 F 2 "" H 2000 2500 50  0001 C CNN
@@
 	2000 2450 2000 2500
 $Comp
-L power:GNDREF #PWR?
+L power:GNDREF #PWR0109
 U 1 1 6087C04F
 P 3850 2450
-F 0 "#PWR?" H 3850 2200 50  0001 C CNN
+F 0 "#PWR0109" H 3850 2200 50  0001 C CNN
 F 1 "GNDREF" H 3855 2277 50  0001 C CNN
 F 2 "" H 3850 2450 50  0001 C CNN
@@
 	3850 2250 3850 2450
 $Comp
-L Device:R R?
+L Device:R R2
 U 1 1 60883081
 P 4100 1650
-F 0 "R?" H 4170 1696 50  0000 L CNN
+F 0 "R2" H 4170 1696 50  0000 L CNN
 F 1 "R" H 4170 1605 50  0000 L CNN
 F 2 "" V 4030 1650 50  0001 C CNN
@@
 	4100 1450 4100 1500
 $Comp
-L Device:LED D?
+L Device:LED D1
 U 1 1 60884984
 P 4100 2000
-F 0 "D?" V 4139 1882 50  0000 R CNN
+F 0 "D1" V 4139 1882 50  0000 R CNN
 F 1 "LED" V 4048 1882 50  0000 R CNN
 F 2 "" H 4100 2000 50  0001 C CNN
@@
 	3850 2200 3850 2250
 $Comp
-L power:+5V #PWR?
+L power:+5V #PWR0110
 U 1 1 608B20C1
 P 4300 1300
-F 0 "#PWR?" H 4300 1150 50  0001 C CNN
+F 0 "#PWR0110" H 4300 1150 50  0001 C CNN
 F 1 "+5V" V 4315 1428 50  0000 L CNN
 F 2 "" H 4300 1300 50  0001 C CNN
@@
 Connection ~ 4100 2200
 $Comp
-L Device:C C?
+L Device:C C5
 U 1 1 608A9FCA
 P 4300 1500
-F 0 "C?" H 4415 1546 50  0000 L CNN
+F 0 "C5" H 4415 1546 50  0000 L CNN
 F 1 "C" H 4415 1455 50  0000 L CNN
 F 2 "Capacitor_SMD:C_1206_3216Metric_Pad1.33x1.80mm_HandSolder" H 4338 1350 50  0001 C CNN
@@
 Connection ~ 4300 1350
 Text GLabel 1800 5050 0    50   Input ~ 0
-Teensy_Uart_RX
+GPS_Uart_RX
 Text GLabel 1800 5150 0    50   Input ~ 0
-Teensy_Uart_TX
+GPS_Uart_TX
 Wire Wire Line
 	1800 5050 2050 5050
@@
 $EndSheet
 $Comp
-L Device:Battery BT?
+L Device:Battery BT1
 U 1 1 60A0D572
 P 800 2500
-F 0 "BT?" H 908 2546 50  0000 L CNN
+F 0 "BT1" H 908 2546 50  0000 L CNN
 F 1 "Battery" H 908 2455 50  0000 L CNN
 F 2 "Connector_PinSocket_2.00mm:PinSocket_1x02_P2.00mm_Vertical" V 800 2560 50  0001 C CNN
@@
 $EndComp
 $Comp
-L power:+BATT #PWR?
+L power:+BATT #PWR0111
 U 1 1 60A138F9
 P 800 2150
-F 0 "#PWR?" H 800 2000 50  0001 C CNN
+F 0 "#PWR0111" H 800 2000 50  0001 C CNN
 F 1 "+BATT" H 815 2323 50  0000 C CNN
 F 2 "" H 800 2150 50  0001 C CNN
@@
 P 800 1050
 AR Path="/6092276E/60A65488" Ref="#PWR?"  Part="1"
-AR Path="/60A65488" Ref="#PWR?"  Part="1"
-F 0 "#PWR?" H 800 900 50  0001 C CNN
+AR Path="/60A65488" Ref="#PWR0112"  Part="1"
+F 0 "#PWR0112" H 800 900 50  0001 C CNN
 F 1 "VCC" H 815 1223 50  0000 C CNN
 F 2 "" H 800 1050 50  0001 C CNN
@@
 $EndComp
 $Comp
-L power:GNDREF #PWR?
+L power:GNDREF #PWR0113
 U 1 1 60A67F58
 P 800 2950
-F 0 "#PWR?" H 800 2700 50  0001 C CNN
+F 0 "#PWR0113" H 800 2700 50  0001 C CNN
 F 1 "GNDREF" H 805 2777 50  0001 C CNN
 F 2 "" H 800 2950 50  0001 C CNN
@@
 $EndComp
 $Comp
-L power:+5V #PWR?
+L power:+5V #PWR0114
 U 1 1 60A6AEA9
 P 2650 4500
-F 0 "#PWR?" H 2650 4350 50  0001 C CNN
+F 0 "#PWR0114" H 2650 4350 50  0001 C CNN
 F 1 "+5V" V 2665 4628 50  0000 L CNN
 F 2 "" H 2650 4500 50  0001 C CNN
@@
 $EndComp
 $Comp
-L power:+3V3 #PWR?
+L power:+3V3 #PWR0115
 U 1 1 60A6C4F6
 P 2950 4500
-F 0 "#PWR?" H 2950 4350 50  0001 C CNN
+F 0 "#PWR0115" H 2950 4350 50  0001 C CNN
 F 1 "+3V3" H 2965 4673 50  0000 C CNN
 F 2 "" H 2950 4500 50  0001 C CNN
@@
 	2950 4600 2950 4650
 $Comp
-L power:GNDREF #PWR?
+L power:GNDREF #PWR0116
 U 1 1 60A746A9
-P 2850 7400
-F 0 "#PWR?" H 2850 7150 50  0001 C CNN
-F 1 "GNDREF" H 2855 7227 50  0001 C CNN
-F 2 "" H 2850 7400 50  0001 C CNN
-F 3 "" H 2850 7400 50  0001 C CNN
-	1    2850 7400
+P 2450 7400
+F 0 "#PWR0116" H 2450 7150 50  0001 C CNN
+F 1 "GNDREF" H 2455 7227 50  0001 C CNN
+F 2 "" H 2450 7400 50  0001 C CNN
+F 3 "" H 2450 7400 50  0001 C CNN
+	1    2450 7400
 	1    0    0    -1
 $EndComp
@@
 	2750 7250 2750 7400
 Connection ~ 2750 7400
-Wire Wire Line
-	2750 7400 2850 7400
 Wire Wire Line
 	2650 7250 2650 7400
@@
 P 4000 5100
 AR Path="/6092276E/60A92742" Ref="R?"  Part="1"
-AR Path="/60A92742" Ref="R?"  Part="1"
-F 0 "R?" H 4070 5146 50  0000 L CNN
+AR Path="/60A92742" Ref="R1"  Part="1"
+F 0 "R1" H 4070 5146 50  0000 L CNN
 F 1 "TBU" H 4070 5055 50  0000 L CNN
 F 2 "Resistor_SMD:R_0603_1608Metric_Pad0.98x0.95mm_HandSolder" V 3930 5100 50  0001 C CNN
@@
 P 4300 5100
 AR Path="/6092276E/60A95088" Ref="R?"  Part="1"
-AR Path="/60A95088" Ref="R?"  Part="1"
-F 0 "R?" H 4370 5146 50  0000 L CNN
+AR Path="/60A95088" Ref="R3"  Part="1"
+F 0 "R3" H 4370 5146 50  0000 L CNN
 F 1 "TBU" H 4370 5055 50  0000 L CNN
 F 2 "Resistor_SMD:R_0603_1608Metric_Pad0.98x0.95mm_HandSolder" V 4230 5100 50  0001 C CNN
@@
 Wire Wire Line
 	3050 4600 3050 4650
-Wire Wire Line
-	4300 4950 4300 4600
-Wire Wire Line
-	4300 4600 4000 4600
-Connection ~ 3050 4600
-Wire Wire Line
-	4000 4950 4000 4600
-Connection ~ 4000 4600
-Wire Wire Line
-	4000 4600 3050 4600
-Text Notes 3600 4500 0    50   ~ 0
+Text Notes 3250 4450 0    50   ~ 0
 Pullups need to be calculated based \non slva689 application note from \ntexas instruments\n
 Wire Wire Line
 	1800 1550 2000 1550
+$Comp
+L power:+3V3 #PWR0117
+U 1 1 60A5C7F9
+P 4150 4850
+F 0 "#PWR0117" H 4150 4700 50  0001 C CNN
+F 1 "+3V3" H 4165 5023 50  0000 C CNN
+F 2 "" H 4150 4850 50  0001 C CNN
+F 3 "" H 4150 4850 50  0001 C CNN
+	1    4150 4850
+	1    0    0    -1
+$EndComp
+Wire Wire Line
+	4000 4950 4000 4900
+Wire Wire Line
+	4000 4900 4150 4900
+Wire Wire Line
+	4150 4900 4150 4850
+Wire Wire Line
+	4300 4950 4300 4900
+Wire Wire Line
+	4300 4900 4150 4900
+Connection ~ 4150 4900
+Connection ~ 2450 7400
+Wire Wire Line
+	2750 7400 2850 7400
 $EndSCHEMATC

Commit message: Added footprints to all componetns
Parts:
- D1: footprint (none) -> Resistor_SMD:R_0603_1608Metric_Pad0.98x0.95mm_HandSolder
- J1: footprint (none) -> Connector_PinHeader_2.54mm:PinHeader_2x20_P2.54mm_Vertical
- R2: value R -> 1k; footprint (none) -> Resistor_SMD:R_0603_1608Metric_Pad0.98x0.95mm_HandSolder
Changed lines of the file:
@@
 F 0 "J1" H 2165 7431 50  0000 C CNN
 F 1 "Raspberry_Pi_2_3" H 2165 7340 50  0000 C CNN
-F 2 "" H 2850 5950 50  0001 C CNN
+F 2 "Connector_PinHeader_2.54mm:PinHeader_2x20_P2.54mm_Vertical" H 2850 5950 50  0001 C CNN
 F 3 "https://www.raspberrypi.org/documentation/hardware/raspberrypi/schematics/rpi_SCH_3bplus_1p0_reduced.pdf" H 2850 5950 50  0001 C CNN
 	1    2850 5950
@@
 P 4100 1650
 F 0 "R2" H 4170 1696 50  0000 L CNN
-F 1 "R" H 4170 1605 50  0000 L CNN
-F 2 "" V 4030 1650 50  0001 C CNN
+F 1 "1k" H 4170 1605 50  0000 L CNN
+F 2 "Resistor_SMD:R_0603_1608Metric_Pad0.98x0.95mm_HandSolder" V 4030 1650 50  0001 C CNN
 F 3 "~" H 4100 1650 50  0001 C CNN
 	1    4100 1650
@@
 F 0 "D1" V 4139 1882 50  0000 R CNN
 F 1 "LED" V 4048 1882 50  0000 R CNN
-F 2 "" H 4100 2000 50  0001 C CNN
+F 2 "Resistor_SMD:R_0603_1608Metric_Pad0.98x0.95mm_HandSolder" H 4100 2000 50  0001 C CNN
 F 3 "~" H 4100 2000 50  0001 C CNN
 	1    4100 2000
